Commit message: added top_plate mesh and switched to .stl format for all meshes

File: mitro/mitro_description/urdf/mitro.urdf.xacro (robot description, xacro)
@@ -7,24 +7,16 @@
     <property name="hokuyo_scan_height" value="0.056"/>
     <macro name="mitro">
+      <link name="base_link">
+      </link>
       <link name="base_plate">
         <visual>
           <origin xyz="0 0 0.0" rpy="0 0 0" />
           <geometry>
-            <mesh filename="package://mitro_description/meshes/base_plate.dae"/>
+            <mesh filename="package://mitro_description/meshes/base_plate.stl"/>
           </geometry>
-          <!--<material name="wood">
-            <texture filename="package://tele_description/meshes/wood.tga"/>
-          </material>-->
+	  <material name="wood">
+	    <color rgba="0.65 0.5 0.37 1"/>
+	  </material>
         </visual>
-      </link>
-      <link name="base_laser">
-        <visual>
-          <origin xyz="0 0 ${-hokuyo_scan_height}" rpy="0 0 0" />
-          <geometry>
-            <mesh filename="package://mitro_description/meshes/hokuyo_urg_2.dae"/>
-          </geometry>
-        </visual>
-      </link>
-      <link name="base_link">
       </link>
       <joint name="base_plate_joint" type="fixed">
@@ -33,4 +25,15 @@
         <child link="base_plate"/>
       </joint>
+      <link name="base_laser">
+	<visual>
+	  <origin xyz="0.0 0.0 ${-hokuyo_scan_height}" rpy="${M_PI/2} 0 ${M_PI/2}" />
+	  <geometry>OD
+	    <mesh filename="package://mitro_description/meshes/hokuyo_urg.stl"/>
+	  </geometry>
+	  <material name="dark grey">
+	    <color rgba="0.2 0.2 0.2 1"/>
+	  </material>
+	</visual>
+      </link>
       <joint name="base_laser_joint" type="fixed">
         <origin xyz="${base_diameter/2 - 0.030 - 0.025} 0.002 ${hokuyo_scan_height + 0.019}" rpy="0 0 -0.032" />
@@ -38,4 +41,36 @@
         <child link="base_laser"/>
       </joint>
+      <link name="top_plate">
+        <visual>
+          <origin xyz="0 0 0.0" rpy="0 0 0" />
+          <geometry>
+            <mesh filename="package://mitro_description/meshes/top_plate.stl"/>
+          </geometry>
+	  <material name="wood">
+	    <color rgba="0.65 0.5 0.37 1"/>
+	  </material>
+        </visual>
+      </link>
+      <joint name="top_plate_joint" type="fixed">
+        <origin xyz="0 0 0.15"/>
+        <parent link="base_plate"/>
+        <child link="top_plate"/>
+      </joint>
+      <link name="kinect_link">
+	<visual>
+	  <origin xyz="0.0 0.0 0.0" rpy="0 0 0" />
+	  <geometry>
+	    <mesh filename="package://mitro_description/meshes/kinect.stl"/>
+	  </geometry>
+	  <material name="dark grey">
+	    <color rgba="0.2 0.2 0.2 1"/>
+	  </material>
+	</visual>
+      </link>
+      <joint name="kinect_joint" type="fixed">
+        <origin xyz="0 0 1.5"/>
+        <parent link="base_link"/>
+        <child link="kinect_link"/>
+      </joint>
     </macro>
     <mitro />

Commit message: included kinect links

File: mitro/mitro_description/urdf/mitro.urdf.xacro (robot description, xacro)
@@ -28,5 +28,5 @@
 	<visual>
 	  <origin xyz="0.0 0.0 ${-hokuyo_scan_height}" rpy="${M_PI/2} 0 ${M_PI/2}" />
-	  <geometry>OD
+	  <geometry>
 	    <mesh filename="package://mitro_description/meshes/hokuyo_urg.stl"/>
 	  </geometry>
@@ -43,5 +43,5 @@
       <link name="top_plate">
         <visual>
-          <origin xyz="0 0 0.0" rpy="0 0 0" />
+          <origin xyz="0 0 0" rpy="0 0 0" />
           <geometry>
             <mesh filename="package://mitro_description/meshes/top_plate.stl"/>
@@ -57,7 +57,8 @@
         <child link="top_plate"/>
       </joint>
+<!-- kinect -->
       <link name="kinect_link">
 	<visual>
-	  <origin xyz="0.0 0.0 0.0" rpy="0 0 0" />
+	  <origin xyz="0 0 0" rpy="0 0 0" />
 	  <geometry>
 	    <mesh filename="package://mitro_description/meshes/kinect.stl"/>
@@ -69,7 +70,31 @@
       </link>
       <joint name="kinect_joint" type="fixed">
-        <origin xyz="0 0 1.5"/>
+        <origin xyz="0 0 1.56" rpy="0 1.16 0"/>
         <parent link="base_link"/>
         <child link="kinect_link"/>
+      </joint>
+      <link name="kinect_depth_frame"/>
+      <joint name="kinect_depth_frame_joint" type="fixed">
+	<origin xyz="0 -0.02 0"/>
+	<parent link="kinect_link"/>
+	<child link="kinect_depth_frame"/>
+      </joint>
+      <link name="kinect_rgb_frame"/>
+      <joint name="kinect_rgb_frame_joint" type="fixed">
+	<origin xyz="0 -0.045 0"/>
+	<parent link="kinect_link"/>
+	<child link="kinect_rgb_frame"/>
+      </joint>
+      <link name="kinect_depth_optical_frame"/>
+      <joint name="kinect_depth_frame_optical_joint" type="fixed">
+	<origin xyz="0 0 0" rpy="-${M_PI/2} 0 -${M_PI/2}"/>
+	<parent link="kinect_depth_frame"/>
+	<child link="kinect_depth_optical_frame"/>
+      </joint>
+      <link name="kinect_rgb_optical_frame"/>
+      <joint name="kinect_rgb_frame_optical_joint" type="fixed">
+	<origin xyz="0 0 0" rpy="-${M_PI/2} 0 -${M_PI/2}"/>
+	<parent link="kinect_rgb_frame"/>
+	<child link="kinect_rgb_optical_frame"/>
       </joint>
     </macro>

Commit message: updated urdf, needs still lots of meassurements

File: mitro/mitro_description/urdf/mitro.urdf.xacro (robot description, xacro)
@@ -4,6 +4,11 @@
     <property name="M_PI" value="3.14159"/>
     <property name="base_diameter" value="0.4572"/>
-    <property name="base_lift" value="0.11"/>
+    <property name="base_plate_lift" value="0.11"/>
+    <property name="base_plate_height" value="0.016"/>
+    <property name="top_plate_lift" value="0.15"/> <!-- TODO: requires meassurement -->
+    <property name="top_plate_height" value="0.016"/> <!-- TODO: requires meassurement -->
     <property name="hokuyo_scan_height" value="0.056"/>
+    <property name="pole_length" value="1.5"/>
+    <property name="kinect_pitch_angle" value="1.16"/>
     <macro name="mitro">
       <link name="base_link">
@@ -11,5 +16,5 @@
       <link name="base_plate">
         <visual>
-          <origin xyz="0 0 0.0" rpy="0 0 0" />
+          <origin xyz="0 0 -${base_plate_height}" rpy="0 0 0" />
           <geometry>
             <mesh filename="package://mitro_description/meshes/base_plate.stl"/>
@@ -21,5 +26,5 @@
       </link>
       <joint name="base_plate_joint" type="fixed">
-        <origin xyz="0 0 ${base_lift}"/>
+        <origin xyz="0 0 ${base_plate_lift}"/>
         <parent link="base_link"/>
         <child link="base_plate"/>
@@ -43,5 +48,5 @@
       <link name="top_plate">
         <visual>
-          <origin xyz="0 0 0" rpy="0 0 0" />
+          <origin xyz="0 0 -${top_plate_height}" rpy="0 0 0" />
           <geometry>
             <mesh filename="package://mitro_description/meshes/top_plate.stl"/>
@@ -53,7 +58,29 @@
       </link>
       <joint name="top_plate_joint" type="fixed">
-        <origin xyz="0 0 0.15"/>
+        <origin xyz="0 0 ${top_plate_lift}"/>
         <parent link="base_plate"/>
         <child link="top_plate"/>
+      </joint>
+      <link name="base_pole_link" />
+      <joint name="base_pole_joint" type="fixed">
+	<origin xyz="-0.05 0 0" rpy="0 0 0"/> <!-- TODO: meassurement required -->
+	<parent link="base_plate"/>
+	<child link="base_pole_link"/>
+      </joint>
+      <link name="top_pole_link">
+        <visual>
+          <origin xyz="0 0 -${pole_length/2}" rpy="0 0 0" />
+          <geometry>
+	    <box size="0.04 0.04 ${pole_length}"/>
+          </geometry>
+	  <material name="aluminium">
+	    <color rgba="0.8 0.8 0.8 1"/>
+	  </material>
+        </visual>
+      </link>
+      <joint name="top_pole_joint" type="fixed">
+	<origin xyz="0 0 ${pole_length}" rpy="0 0 0"/>
+	<parent link="base_pole_link"/>
+	<child link="top_pole_link"/>
       </joint>
 <!-- kinect -->
@@ -70,6 +97,6 @@
       </link>
       <joint name="kinect_joint" type="fixed">
-        <origin xyz="0 0 1.56" rpy="0 1.16 0"/>
-        <parent link="base_link"/>
+        <origin xyz="0.1 0 0" rpy="0 ${kinect_pitch_angle} 0"/> <!-- TODO: requires meassurement -->
+        <parent link="top_pole_link"/>
         <child link="kinect_link"/>
       </joint>

Commit message: changed a few dimensions/messurements

File: mitro/mitro_description/urdf/mitro.urdf.xacro (robot description, xacro)
@@ -6,8 +6,9 @@
     <property name="base_plate_lift" value="0.11"/>
     <property name="base_plate_height" value="0.016"/>
-    <property name="top_plate_lift" value="0.15"/> <!-- TODO: requires meassurement -->
+    <property name="top_plate_lift" value="0.12"/>
     <property name="top_plate_height" value="0.016"/> <!-- TODO: requires meassurement -->
     <property name="hokuyo_scan_height" value="0.056"/>
-    <property name="pole_length" value="1.5"/>
+    <property name="pole_length" value="1.45"/>
+    <property name="pole_x_offset" value="-0.0611"/>
     <property name="kinect_pitch_angle" value="1.16"/>
     <macro name="mitro">
@@ -64,5 +65,5 @@
       <link name="base_pole_link" />
       <joint name="base_pole_joint" type="fixed">
-	<origin xyz="-0.05 0 0" rpy="0 0 0"/> <!-- TODO: meassurement required -->
+	<origin xyz="${pole_x_offset} 0 0" rpy="0 0 0"/>
 	<parent link="base_plate"/>
 	<child link="base_pole_link"/>
@@ -72,5 +73,5 @@
           <origin xyz="0 0 -${pole_length/2}" rpy="0 0 0" />
           <geometry>
-	    <box size="0.04 0.04 ${pole_length}"/>
+	    <box size="0.045 0.045 ${pole_length}"/>
           </geometry>
 	  <material name="aluminium">
@@ -97,5 +98,5 @@
       </link>
       <joint name="kinect_joint" type="fixed">
-        <origin xyz="0.1 0 0" rpy="0 ${kinect_pitch_angle} 0"/> <!-- TODO: requires meassurement -->
+        <origin xyz="0.095 -0.01 0" rpy="0 ${kinect_pitch_angle} 0"/> <!-- TODO: requires meassurement -->
         <parent link="top_pole_link"/>
         <child link="kinect_link"/>
@@ -103,5 +104,5 @@
       <link name="kinect_depth_frame"/>
       <joint name="kinect_depth_frame_joint" type="fixed">
-	<origin xyz="0 -0.02 0"/>
+	<origin xyz="0 0.0125 0"/>
 	<parent link="kinect_link"/>
 	<child link="kinect_depth_frame"/>
@@ -109,5 +110,5 @@
       <link name="kinect_rgb_frame"/>
       <joint name="kinect_rgb_frame_joint" type="fixed">
-	<origin xyz="0 -0.045 0"/>
+	<origin xyz="0 0.0125 0"/>
 	<parent link="kinect_link"/>
 	<child link="kinect_rgb_frame"/>

Commit message: recalibrated kinect link

File: mitro/mitro_description/urdf/mitro.urdf.xacro (robot description, xacro)
@@ -88,5 +88,5 @@
       <link name="kinect_link">
 	<visual>
-	  <origin xyz="0 0 0" rpy="0 0 0" />
+	  <origin xyz="0 0.01 0" rpy="0 0 0" />
 	  <geometry>
 	    <mesh filename="package://mitro_description/meshes/kinect.stl"/>
@@ -98,5 +98,5 @@
       </link>
       <joint name="kinect_joint" type="fixed">
-        <origin xyz="0.095 -0.01 0" rpy="0 ${kinect_pitch_angle} 0"/> <!-- TODO: requires meassurement -->
+        <origin xyz="0.08 -0.01 0" rpy="0 ${kinect_pitch_angle} 0"/> <!-- TODO: requires meassurement -->
         <parent link="top_pole_link"/>
         <child link="kinect_link"/>

Commit message: urdf update for sonar link

File: mitro/mitro_description/urdf/mitro.urdf.xacro (robot description, xacro)
@@ -9,4 +9,5 @@
     <property name="top_plate_height" value="0.016"/> <!-- TODO: requires meassurement -->
     <property name="hokuyo_scan_height" value="0.056"/>
+    <property name="sonar_scan_height" value="0.035"/>
     <property name="pole_length" value="1.45"/>
     <property name="pole_x_offset" value="-0.0611"/>
@@ -30,4 +31,11 @@
         <parent link="base_link"/>
         <child link="base_plate"/>
+      </joint>
+      <link name="base_sonar">
+      </link>
+      <joint name="base_sonar_joint" type="fixed">
+        <origin xyz="0 0 ${sonar_scan_height}"/>
+        <parent link="base_plate"/>
+        <child link="base_sonar"/>
       </joint>
       <link name="base_laser">

Commit message: sort-of calibrated urdf file

File: mitro/mitro_description/urdf/mitro.urdf.xacro (robot description, xacro)
@@ -2,15 +2,17 @@
 <robot name="mitro">
     <!-- Properties (Constants) -->
-    <property name="M_PI" value="3.14159"/>
+    <property name="M_PI" value="3.14159265359"/>
     <property name="base_diameter" value="0.4572"/>
-    <property name="base_plate_lift" value="0.11"/>
-    <property name="base_plate_height" value="0.016"/>
-    <property name="top_plate_lift" value="0.12"/>
-    <property name="top_plate_height" value="0.016"/> <!-- TODO: requires meassurement -->
+    <property name="base_plate_lift" value="0.112"/> <!-- lift top top of plate -->
+    <property name="base_plate_height" value="0.0123"/>
+    <property name="top_plate_lift" value="0.121"/> <!-- lift to top of plate -->
+    <property name="top_plate_height" value="0.0066"/>
     <property name="hokuyo_scan_height" value="0.056"/>
-    <property name="sonar_scan_height" value="0.035"/>
+    <property name="sonar_scan_height" value="0.037"/>
     <property name="pole_length" value="1.45"/>
     <property name="pole_x_offset" value="-0.0611"/>
-    <property name="kinect_pitch_angle" value="1.27"/>
+    <property name="kinect_pitch_angle" value="1.18"/>
+    <property name="kinect_roll_angle" value="0.04"/>
+    <property name="kinect_yaw_angle" value="0.0"/>
     <macro name="mitro">
       <link name="base_link">
@@ -51,5 +53,5 @@
       </link>
       <joint name="base_laser_joint" type="fixed">
-        <origin xyz="${base_diameter/2 - 0.030 - 0.025} 0.002 ${hokuyo_scan_height + 0.019}" rpy="0 0 -0.032" />
+        <origin xyz="${base_diameter/2 - 0.030 - 0.025} 0.002 ${hokuyo_scan_height + 0.021}" rpy="0 0 -0.032" />
         <parent link="base_plate"/>
         <child link="base_laser"/>
@@ -96,5 +98,5 @@
       <link name="kinect_link">
 	<visual>
-	  <origin xyz="0 0.01 0" rpy="0 0 0" />
+	  <origin xyz="0 0 0" rpy="0 0 0" />
 	  <geometry>
 	    <mesh filename="package://mitro_description/meshes/kinect.stl"/>
@@ -106,5 +108,5 @@
       </link>
       <joint name="kinect_joint" type="fixed">
-        <origin xyz="0.08 -0.01 0" rpy="0 ${kinect_pitch_angle} 0"/> <!-- TODO: requires meassurement -->
+        <origin xyz="0.10 -0.04 0" rpy="${kinect_roll_angle} ${kinect_pitch_angle} ${kinect_yaw_angle}"/> <!-- TODO: requires meassurement -->
         <parent link="top_pole_link"/>
         <child link="kinect_link"/>
@@ -112,5 +114,5 @@
       <link name="kinect_depth_frame"/>
       <joint name="kinect_depth_frame_joint" type="fixed">
-	<origin xyz="0 0.0125 0"/>
+	<origin xyz="0 0.049 0"/>
 	<parent link="kinect_link"/>
 	<child link="kinect_depth_frame"/>
@@ -118,5 +120,5 @@
       <link name="kinect_rgb_frame"/>
       <joint name="kinect_rgb_frame_joint" type="fixed">
-	<origin xyz="0 0.0125 0"/>
+	<origin xyz="0 0.022 0"/>
 	<parent link="kinect_link"/>
 	<child link="kinect_rgb_frame"/>

Commit message: some more urdf fine-tuning

File: mitro/mitro_description/urdf/mitro.urdf.xacro (robot description, xacro)
@@ -13,6 +13,6 @@
     <property name="pole_x_offset" value="-0.0611"/>
     <property name="kinect_pitch_angle" value="1.18"/>
-    <property name="kinect_roll_angle" value="0.04"/>
-    <property name="kinect_yaw_angle" value="0.0"/>
+    <property name="kinect_roll_angle" value="0.06"/>
+    <property name="kinect_yaw_angle" value="0.02"/>
     <macro name="mitro">
       <link name="base_link">
@@ -96,5 +96,5 @@
       </joint>
 <!-- kinect -->
-      <link name="kinect_link">
+      <link name="kinect_model_link">
 	<visual>
 	  <origin xyz="0 0 0" rpy="0 0 0" />
@@ -107,6 +107,12 @@
 	</visual>
       </link>
+      <joint name="kinect_model_joint" type="fixed">
+        <origin xyz="0.10 0 0" rpy="0 ${kinect_pitch_angle} 0"/>
+        <parent link="top_pole_link"/>
+        <child link="kinect_model_link"/>
+      </joint>
+      <link name="kinect_link"/>
       <joint name="kinect_joint" type="fixed">
-        <origin xyz="0.10 -0.04 0" rpy="${kinect_roll_angle} ${kinect_pitch_angle} ${kinect_yaw_angle}"/> <!-- TODO: requires meassurement -->
+        <origin xyz="0.10 -0.06 0" rpy="${kinect_roll_angle} ${kinect_pitch_angle} ${kinect_yaw_angle}"/> <!-- TODO: requires meassurement -->
         <parent link="top_pole_link"/>
         <child link="kinect_link"/>

Commit message: urdf kinect tweak

File: mitro/mitro_description/urdf/mitro.urdf.xacro (robot description, xacro)
@@ -114,5 +114,5 @@
       <link name="kinect_link"/>
       <joint name="kinect_joint" type="fixed">
-        <origin xyz="0.10 -0.06 0" rpy="${kinect_roll_angle} ${kinect_pitch_angle} ${kinect_yaw_angle}"/> <!-- TODO: requires meassurement -->
+        <origin xyz="0.11 -0.08 0" rpy="${kinect_roll_angle} ${kinect_pitch_angle} ${kinect_yaw_angle}"/> <!-- TODO: requires meassurement -->
         <parent link="top_pole_link"/>
         <child link="kinect_link"/>
